File: recieving end copy-1.brd (EAGLE design)
At the start: 57.8 x 64.5 mm, 38 parts, among them IC1 MEGA8-P

Commit message: in the transmission end, we fixed the design for the transistors for the diodes and the input signal, so it operates with PMOS transistors the way we want it. In the receiving end, we fixed the design for the transistor and just decided to use an NOMS transistors, and it is working the way we want it. Now that both ends are working and tested. we need to merge them in one file to submit the one file to sunstone
Parts:
- removed T1, T2: (no value), solomon_library:SOT-23
- added Q1, Q2: BSS295, transistor-fet:TO92
- moved R20 5.24 mm to (28.2, 40.6), turned to 270 degrees
- moved R21 2.03 mm to (32.5, 33.3), turned to 180 degrees
- moved C4 0.51 mm to (32.0, 29.5)
Connections:
- net GND: now also Q1.2, Q2.2; no longer T1.1, T2.1
- net LED1-: now also Q1.3; no longer T2.2
- net LED2-: now also Q2.3; no longer T1.2
- net N$1: now also Q1.1; no longer T2.3
- net N$8: now also Q2.1; no longer T1.3
Routing:
- net N$8: track 22.4 -> 12.4 mm
- net N$1: track 34.8 -> 27.2 mm, vias 3 -> 1
- net N$9: track 82.3 -> 87.4 mm
- net LED1-: track 32.2 -> 30.0 mm, vias 1 -> 0
- net LED2-: track 21.0 -> 19.3 mm, vias 2 -> 0
- net N$41: track 22.8 -> 23.6 mm
Other:
- board size 57.8 x 64.5 mm -> 57.9 x 64.3 mm
